File: Mk1/Electronics/MK1.kicad_sch (KiCad schematic)
At the start: 121 parts, among them SW1 SW_Push, SW10 SW_Push, SW11 SW_Push, SW12 SW_Push, SW13 SW_Push, SW14 SW_Push, SW15 SW_Push, SW16 SW_Push, SW17 SW_Push, SW18 SW_Push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

Commit message: Move Mk1 electronics to Mk1 directory.
Other:
- title: Keyboard Mk2 -> Keyboard Mk1
Changed lines of the file:
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@@
   (paper "A4")
   (title_block
-    (title "Keyboard Mk2")
+    (title "Keyboard Mk1")
     (rev "1")
   )
